File: C810_New!.kicad_pcb (KiCad board)
At the start: 2 copper layers, 90 x 60 mm, 121 parts, among them J1 Conn_01x02_Pin, J10 V_High, J11 W_Low, J12 W_High, J13 V_Low, J14 U_Low, J15 5V, J16 3.3V, J17 12V, J18 Screw_Terminal_01x03, J19 24V, J2 Conn_01x04, J20 GND, J21 GND, J22 GND, J23 GND, J3 Conn_ST_STDC14, J4 USB_C_Receptacle_USB2.0_16P, J5 test, J6 U_current, J7 V_current, J8 W_current, J9 U_High, Q1 BSC159N10LSFG, Q2 BSC159N10LSFG, Q3 BSC159N10LSFG, Q4 BSC159N10LSFG, Q5 BSC159N10LSFG, Q6 BSC159N10LSFG, SW1 Reset, U1 IR2302, U10 L7812, U11 Regulator_3.3, U12 Regulator_5.0, U2 IR2302, U3 IR2302, U4 STM32F303K8Tx, U5 NCS214, U6 NCS214, U7 NCS214, U8 MCP2561-E-SN, Y1 16MHz

Commit message: M3508用のGHコネクタを追加
PCBの配線し直し開始
Parts:
- removed J21, J22: GND, Connector_PinHeader_1.00mm:PinHeader_1x01_P1.00mm_Vertical
- C20: value 2.2μ -> 1μ
- J20: value GND -> Conn_01x07; footprint Connector_PinHeader_1.00mm:PinHeader_1x01_P1.00mm_Vertical -> Connector_JST:JST_GH_SM07B-GHS-TB_1x07-1MP_P1.25mm_Horizontal
- moved Q3 80.7 mm to (57.5, 128.2)
- moved D3 80.7 mm to (53.0, 122.6)
- moved D6 80.7 mm to (45.7, 128.8)
- moved Q4 80.7 mm to (49.8, 127.4)
- moved G*** 76.2 mm to (232.0, 68.3)
- moved J20 75.2 mm to (84.6, 105.1)
- moved C14 68.7 mm to (140.7, 147.4)
- moved J8 68.7 mm to (144.5, 144.9)
- moved R19 68.7 mm to (134.9, 139.8)
- moved R21 68.7 mm to (138.3, 141.1)
- moved U7 68.7 mm to (140.4, 144.3)
- moved C12 68.7 mm to (140.4, 140.4)
- moved R20 68.7 mm to (138.4, 139.6)
- moved R25 68.7 mm to (143.2, 147.9)
- moved R15 59.1 mm to (112.2, 141.7)
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Connections:
- D5 pad 2: GND -> U_L_Side
- D6 pad 2: GND -> V_L_Side
- D9 pad 2: GND -> W_L_Side
- J20 pad 1: GND -> unconnected-(J20-Pin_1-Pad1)
- Q2 pad 1: GND -> U_L_Side
- Q2 pad 2: GND -> U_L_Side
- Q2 pad 3: GND -> U_L_Side
- Q4 pad 1: GND -> V_L_Side
- Q4 pad 2: GND -> V_L_Side
- Q4 pad 3: GND -> V_L_Side
- Q6 pad 1: GND -> W_L_Side
- Q6 pad 2: GND -> W_L_Side
- Q6 pad 3: GND -> W_L_Side
- R12 pad 2: GND -> W_L_Side
- R13 pad 1: +24V -> U_L_Side
- R13 pad 2: U_H_Side -> GND
- R14 pad 1: +24V -> V_L_Side
- R14 pad 2: V_H_Side -> GND
- R15 pad 1: +24V -> V_L_Side
- R16 pad 1: +24V -> U_L_Side
- R17 pad 1: U_H_Side -> GND
- R18 pad 1: V_H_Side -> GND
- R19 pad 1: +24V -> W_L_Side
- R19 pad 2: W_H_Side -> GND
- R20 pad 1: +24V -> W_L_Side
- R21 pad 1: W_H_Side -> GND
- R3 pad 2: GND -> U_L_Side
- R8 pad 2: GND -> V_L_Side
Routing:
- net U_Current: track 47.8 -> 33.2 mm
- net +24V: track 22.0 -> 7.55 mm
- net V_Current: track 44.0 -> 29.6 mm, vias 2 -> 1
- net W_Current: track 55.2 -> 41.0 mm, vias 2 -> 1
- net +3.3V: track 234.6 -> 228.8 mm, vias 7 -> 4
- net Net-(U5-+IN): track 5.13 -> 0.00 mm
- net Net-(U7-+IN): track 5.07 -> 0.00 mm
- net Net-(U6-+IN): track 4.99 -> 0.00 mm
- net V_H_Side: track 3.90 -> 0.00 mm
- net W_H_Side: track 3.82 -> 0.00 mm
- net U_H_Side: track 3.73 -> 0.00 mm
- net Net-(U5--IN): track 3.18 -> 0.00 mm
- net Net-(U7--IN): track 3.12 -> 0.00 mm
- net Net-(U6--IN): track 3.01 -> 0.00 mm
- net W_OUT: track 29.1 -> 28.2 mm, vias 2 -> 1
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- removed copper zone on F.Cu, net +24V
- removed copper zone on B.Cu, net GND
- removed copper zone on F.Cu, net GND
- removed copper zone on F.Cu, net U_H_Side
- removed copper zone on F.Cu, net U_OUT
- removed copper zone on F.Cu, net V_H_Side
- removed copper zone on F.Cu, net V_OUT
- removed copper zone on F.Cu, net W_H_Side
- removed copper zone on F.Cu, net W_OUT

Commit message: 配線全削除
Parts:
- removed J10: V_High, Connector_PinHeader_1.00mm:PinHeader_1x01_P1.00mm_Vertical
- removed J11: W_Low, Connector_PinHeader_1.00mm:PinHeader_1x01_P1.00mm_Vertical
- removed J12: W_High, Connector_PinHeader_1.00mm:PinHeader_1x01_P1.00mm_Vertical
- removed J13: V_Low, Connector_PinHeader_1.00mm:PinHeader_1x01_P1.00mm_Vertical
- removed J14: U_Low, Connector_PinHeader_1.00mm:PinHeader_1x01_P1.00mm_Vertical
- removed J15: 5V, Connector_PinHeader_1.00mm:PinHeader_1x01_P1.00mm_Vertical
- removed J16: 3.3V, Connector_PinHeader_1.00mm:PinHeader_1x01_P1.00mm_Vertical
- removed J17: 12V, Connector_PinHeader_1.00mm:PinHeader_1x01_P1.00mm_Vertical
- removed J23: GND, Connector_PinHeader_1.00mm:PinHeader_1x01_P1.00mm_Vertical
- removed J6: U_current, TestPoint:TestPoint_Pad_D1.5mm
- removed J7: V_current, TestPoint:TestPoint_Pad_D1.5mm
- removed J8: W_current, TestPoint:TestPoint_Pad_D1.5mm
- removed J9: U_High, Connector_PinHeader_1.00mm:PinHeader_1x01_P1.00mm_Vertical
- added R33: 10k, Resistor_SMD:R_0603_1608Metric, F.Cu at (181.0, 85.3)
- J5: footprint Connector_PinHeader_1.00mm:PinHeader_1x01_P1.00mm_Vertical -> Connector_PinHeader_2.54mm:PinHeader_1x01_P2.54mm_Vertical
- SW1: value Reset -> button
- moved J18 31.3 mm to (82.5, 90.7)
- moved J5 3.42 mm to (183.5, 97.5)
Connections:
- SW1 pad 1: GND -> Net-(U4-PA15)
- SW1 pad 2: NRST -> +3.3V
- U4 pad 25: unconnected-(U4-PA15-Pad25) -> Net-(U4-PA15)
Routing:
- net +3.3V: track 228.8 -> 0.00 mm, vias 4 -> 0
- net +12V: track 127.3 -> 0.00 mm, vias 2 -> 0
- net Encoder_1: track 75.8 -> 0.00 mm, vias 2 -> 0
- net Encoder_2: track 74.8 -> 0.00 mm, vias 2 -> 0
- net NRST: track 55.4 -> 0.00 mm, vias 1 -> 0
- net W_Current: track 41.0 -> 0.00 mm, vias 1 -> 0
- net U_Current: track 33.2 -> 0.00 mm, vias 2 -> 0
- net V_Current: track 29.6 -> 0.00 mm, vias 1 -> 0
- net U_OUT: track 28.6 -> 0.00 mm, vias 1 -> 0
- net W_OUT: track 28.2 -> 0.00 mm, vias 1 -> 0
- net V_OUT: track 28.2 -> 0.00 mm, vias 1 -> 0
- net Net-(Q6-G): track 26.1 -> 0.00 mm, vias 1 -> 0
- net Net-(Q4-G): track 26.0 -> 0.00 mm, vias 1 -> 0
- net Net-(Q2-G): track 25.7 -> 0.00 mm, vias 1 -> 0
- net W_PWM: track 22.7 -> 0.00 mm
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Other:
- board outline removed
- board text added: "BLDC Motor Driver 【C810_Re:New】 ver:1.1"
- board text added: "designed by Watanabe"
- board text removed: "BLDC Motor Driver 【C810_Re:New】 ver:1.0"
- board text removed: "made by Watanabe"

Commit message: C610と同じサイズは無理すぎ
Parts:
- removed the G*** at (134.8, 84.6)
- removed the G*** at (185.0, 98.5)
- removed the G*** at (169.3, 76.2)
- removed the G*** at (134.9, 105.6)
- removed the G*** at (155.8, 103.5)
- removed the G*** at (121.4, 105.7)
- removed H4, H5, H6, H7: M3, MountingHole:MountingHole_3.2mm_M3_Pad_Via
- removed J18: Screw_Terminal_01x03, TerminalBlock:TerminalBlock_bornier-3_P5.08mm
- removed J19: 24V, Connector_PinHeader_1.00mm:PinHeader_1x01_P1.00mm_Vertical
- removed Y1: 16MHz, Crystal:Crystal_HC18-U_Vertical
- added R34: 10k, Resistor_SMD:R_0603_1608Metric, F.Cu at (123.3, 163.8)
- added R35: 10k, Resistor_SMD:R_0603_1608Metric, F.Cu at (123.3, 166.3)
- added R36: 10k, Resistor_SMD:R_0603_1608Metric, F.Cu at (123.3, 168.8)
- added R37: 10k, Resistor_SMD:R_0603_1608Metric, F.Cu at (123.3, 171.3)
- added R38: 10k, Resistor_SMD:R_0603_1608Metric, F.Cu at (123.3, 173.8)
- added R39: 10k, Resistor_SMD:R_0603_1608Metric, F.Cu at (123.3, 176.3)
- added Y2: 16MHz, Crystal:Crystal_SMD_3225-4Pin_3.2x2.5mm_HandSoldering, F.Cu at (158.4, 111.4)
- C10, C17, J20, R16, R17, R23, U5: moved to B.Cu
- J1: value Conn_01x02_Pin -> Conn_01x03; footprint Connector_AMASS:AMASS_XT60PW-M_1x02_P7.20mm_Horizontal -> footprints:MR30; moved to B.Cu
- U11: value Regulator_3.3 -> 3.3
- moved J1 104.8 mm to (89.2, 104.9)
- moved U11 76.3 mm to (119.0, 114.2), turned to -90 degrees
- moved C21 74.6 mm to (110.8, 122.8), turned to 90 degrees
- moved C20 73.0 mm to (112.5, 122.8), turned to 90 degrees
- moved SW1 72.1 mm to (109.0, 111.9), turned to 30 degrees
- moved C24 71.6 mm to (118.1, 109.3), turned to -90 degrees
- moved U4 71.4 mm to (109.3, 137.6)
- moved C23 70.3 mm to (119.6, 109.2), turned to -90 degrees
- moved U10 69.8 mm to (126.2, 109.2), turned to -90 degrees
- moved J4 69.6 mm to (123.8, 122.5)
- moved U8 69.5 mm to (119.1, 121.7)
- moved U12 68.5 mm to (111.8, 117.9), turned to 90 degrees
- moved C19 64.8 mm to (125.4, 104.3), turned to -90 degrees
- moved U5 56.5 mm to (81.9, 94.7), turned to 180 degrees
- moved D6 54.0 mm to (98.0, 115.4), turned to 180 degrees
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Connections:
- J1 pad 1: GND -> U_OUT
- J1 pad 2: +24V -> V_OUT
- J4 pad A1: unconnected-(J4-GND-PadA1)_2 -> GND
- J4 pad A12: unconnected-(J4-GND-PadA1)_3 -> GND
- J4 pad A4: unconnected-(J4-VBUS-PadA4)_1 -> +24V
- J4 pad A9: unconnected-(J4-VBUS-PadA4)_3 -> +24V
- J4 pad B1: unconnected-(J4-GND-PadA1)_1 -> GND
- J4 pad B12: unconnected-(J4-GND-PadA1) -> GND
- J4 pad B4: unconnected-(J4-VBUS-PadA4)_2 -> +24V
- J4 pad B9: unconnected-(J4-VBUS-PadA4) -> +24V
- U5 pad 1: GND -> Net-(U5-REF)
- U6 pad 1: GND -> Net-(U6-REF)
- U7 pad 1: GND -> Net-(U7-REF)
Other:
- board outline added: 44.8 x 23.5 mm
- board text removed: "U"
- board text removed: "V"
- board text removed: "W"

Commit message: あたおかレイアウトを考えてる
Parts:
- removed C10, C12, C7: 1μ, Capacitor_SMD:C_0603_1608Metric
- removed C14: 0.1μ, Capacitor_SMD:C_0603_1608Metric_Pad1.08x0.95mm_HandSolder
- removed J5: test, Connector_PinHeader_2.54mm:PinHeader_1x01_P2.54mm_Vertical
- removed R15, R16, R17, R18, R20, R21: 10, Resistor_SMD:R_0603_1608Metric
- removed R19: 0.5m, Resistor_SMD:R_2512_6332Metric
- removed R23, R24, R25, R26, R27, R28, R38, R39: 10k, Resistor_SMD:R_0603_1608Metric
- removed U7: NCS214, Package_TO_SOT_SMD:SOT-363_SC-70-6_Handsoldering
- C1, C15, C16, C18, C2, C25, C26, C3, C4, C5, C6, D1, D2, D7, FB1, R1, R10, R11, R12, R2, R22, R3, R33, R4, R5, R6, R7, R8, R9, U1, U10, U2, U3, U4: moved to B.Cu
- C11: footprint Capacitor_SMD:C_0603_1608Metric_Pad1.08x0.95mm_HandSolder -> Capacitor_SMD:C_0603_1608Metric
- C17: footprint Capacitor_SMD:C_0603_1608Metric_Pad1.08x0.95mm_HandSolder -> Capacitor_SMD:C_0603_1608Metric; moved to F.Cu
- C22: footprint Capacitor_THT:CP_Radial_D12.5mm_P5.00mm -> Capacitor_SMD:CP_Elec_6.3x7.7
- SW1: footprint Button_Switch_THT:SW_PUSH_1P1T_6x3.5mm_H5.0_APEM_MJTP1250 -> Button_Switch_SMD:SW_Push_1P1T_NO_Vertical_Wuerth_434133025816
- U5: moved to F.Cu
- Y2: footprint Crystal:Crystal_SMD_3225-4Pin_3.2x2.5mm_HandSoldering -> Crystal:Crystal_SMD_3225-4Pin_3.2x2.5mm; moved to B.Cu
- moved R1 77.9 mm to (65.9, 130.8), turned to 180 degrees
- moved R3 77.8 mm to (65.9, 132.2), turned to 180 degrees
- moved C1 76.8 mm to (69.6, 131.5), turned to -90 degrees
- moved R2 75.8 mm to (68.1, 131.5), turned to -90 degrees
- moved R4 74.8 mm to (68.9, 133.8)
- moved R37 72.9 mm to (90.7, 106.0), turned to 90 degrees
- moved LED1 70.2 mm to (110.5, 103.3), turned to 90 degrees
- moved R36 69.4 mm to (89.7, 108.1), turned to 180 degrees
- moved U3 67.7 mm to (100.2, 151.0)
- moved R32 65.7 mm to (109.3, 107.3), turned to 90 degrees
- moved R31 64.8 mm to (110.5, 107.3), turned to 90 degrees
- moved R30 64.1 mm to (111.8, 107.2), turned to 90 degrees
- moved D10 63.9 mm to (117.4, 106.9)
- moved R29 62.8 mm to (114.1, 106.9)
- moved C11 62.1 mm to (92.0, 114.0), turned to -90 degrees
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Connections:
- D3 pad 1: V_H_Side -> +24V
- D4 pad 1: U_H_Side -> +24V
- D8 pad 1: W_H_Side -> +24V
- D9 pad 2: W_L_Side -> GND
- Q1 pad 5: U_H_Side -> +24V
- Q3 pad 5: V_H_Side -> +24V
- Q5 pad 5: W_H_Side -> +24V
- Q6 pad 1: W_L_Side -> GND
- Q6 pad 2: W_L_Side -> GND
- Q6 pad 3: W_L_Side -> GND
- R12 pad 2: W_L_Side -> GND
- U4 pad 30: Net-(J5-Pin_1) -> unconnected-(U4-PB7-Pad30)
- U4 pad 6: W_Current -> unconnected-(U4-PA0-Pad6)
- U5 pad 4: Net-(U5-+IN) -> U_L_Side
- U5 pad 5: Net-(U5--IN) -> GND
- U6 pad 4: Net-(U6-+IN) -> V_L_Side
- U6 pad 5: Net-(U6--IN) -> GND
Routing:
- net +24V: track 0.00 -> 7.95 mm, vias 0 -> 25
- net CAN_L: track 0.00 -> 1.70 mm
- net CAN_H: track 0.00 -> 1.70 mm
- net W_OUT: vias 0 -> 4
- net V_OUT: vias 0 -> 10
- net U_OUT: vias 0 -> 12
- net +12V: vias 0 -> 1
- added copper zone on B.Cu, net +24V
- added copper zone on F.Cu, net +24V
- added copper zone on F.Cu, net U_L_Side
- added copper zone on B.Cu, net U_OUT
- added copper zone on F.Cu, net U_OUT
- added copper zone on F.Cu, net V_L_Side
- added copper zone on B.Cu, net V_OUT
- added copper zone on F.Cu, net V_OUT
- added copper zone on B.Cu, net W_OUT
- added copper zone on F.Cu, net W_OUT

Commit message: 配線が無理すぎるので寝る
Parts:
- R12, R3, R33, R8: moved to F.Cu
- moved R1 44.5 mm to (102.0, 104.8), turned to 90 degrees
- moved R2 41.7 mm to (99.3, 103.8), turned to 0 degrees
- moved C1 39.7 mm to (99.3, 105.1), turned to 180 degrees
- moved C4 39.0 mm to (104.3, 109.8), turned to 90 degrees
- moved R4 38.1 mm to (95.2, 106.2), turned to 90 degrees
- moved U1 37.2 mm to (98.7, 109.2), turned to 90 degrees
- moved R3 35.1 mm to (91.5, 108.2)
- moved C5 34.9 mm to (107.8, 114.3), turned to -90 degrees
- moved R5 34.4 mm to (97.8, 114.5)
- moved C2 34.4 mm to (99.3, 114.5)
- moved R6 34.2 mm to (98.6, 117.3)
- moved C6 33.3 mm to (110.9, 121.4), turned to -90 degrees
- moved FB1 30.3 mm to (110.1, 118.9)
- moved C25 30.2 mm to (118.2, 122.6), turned to 0 degrees
- moved U2 30.0 mm to (103.5, 115.6)
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Connections:
- U4 pad 10: Encoder_1 -> Encoder_2
- U4 pad 11: Encoder_2 -> Encoder_1
- U4 pad 7: V_Current -> U_Current
- U4 pad 8: U_Current -> V_Current
Routing:
- net +3.3V: track 0.00 -> 115.0 mm, vias 0 -> 5
- net U_Current: track 0.00 -> 47.0 mm, vias 0 -> 1
- net +12V: track 0.00 -> 43.9 mm, vias 1 -> 7
- net V_Current: track 0.00 -> 37.3 mm, vias 0 -> 1
- net Encoder_1: track 0.00 -> 32.4 mm, vias 0 -> 1
- net Encoder_2: track 0.00 -> 30.8 mm, vias 0 -> 1
- net U_SD: track 0.00 -> 29.2 mm
- net NRST: track 0.00 -> 25.5 mm, vias 0 -> 1
- net SWO: track 0.00 -> 23.3 mm, vias 0 -> 1
- net Net-(U4-PA15): track 0.00 -> 22.4 mm, vias 0 -> 3
- net SWDIO: track 0.00 -> 20.5 mm, vias 0 -> 1
- net SWCLK: track 0.00 -> 20.3 mm, vias 0 -> 1
- net W_PWM: track 0.00 -> 19.0 mm, vias 0 -> 2
- net U_PWM: track 0.00 -> 18.9 mm, vias 0 -> 2
- net CAN_RX: track 0.00 -> 16.6 mm, vias 0 -> 1
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- added copper zone on B.Cu, net GND
- added copper zone on F.Cu, net GND

Commit message: gomimimimi
Parts:
- moved C27 3.65 mm to (117.4, 107.4)
- moved J1 0.60 mm to (90.7, 103.4)
- moved D10 0.52 mm to (117.4, 106.3)
- moved J4 0.41 mm to (123.9, 122.1)
- moved R13 0.20 mm to (89.0, 102.8)
- moved LED1 0.19 mm to (110.5, 103.5)
- moved R10 0.19 mm to (99.7, 123.6)
Routing:
- net +3.3V: track 115.0 -> 109.7 mm, vias 5 -> 7
- net V_OUT: track 2.11 -> 6.49 mm, vias 11 -> 10
- net CAN_H: track 4.45 -> 5.31 mm
- net V_PWM: track 10.8 -> 11.5 mm
- net U_Current: track 47.0 -> 47.8 mm
- net Encoder_1: track 32.4 -> 32.9 mm
- net U_SD: track 29.2 -> 28.7 mm
- net +24V: track 11.0 -> 11.5 mm, vias 26 -> 24
- net Net-(U2-HO): track 3.75 -> 4.25 mm
- net Net-(U4-PA15): track 22.4 -> 22.0 mm, vias 3 -> 2
- net W_OUT: vias 7 -> 8
- net GND: vias 6 -> 29

Commit message: 配線完了
Parts:
- removed D10: LED, LED_SMD:LED_0603_1608Metric_Pad1.05x0.95mm_HandSolder
- removed R29: 100, Resistor_SMD:R_0603_1608Metric
Routing:
- net +12V: track 43.9 -> 58.8 mm
- net +3.3V: track 109.7 -> 113.4 mm
- net Net-(D10-K): track 1.68 -> 0.00 mm
- net VCP_RX: track 8.58 -> 9.46 mm
- net GND: vias 29 -> 31
- net +24V: vias 24 -> 28
